Commit message: added orbslam2

File: urdf/garry.urdf (robot description, URDF)
Before this commit: robot garry, 4 links, 3 joints
Links:
- link base_link: geometry collision box size=250.0 170. 1.25; visual box size=250.0 170.0 1.25
